File: BKM-10Rp2040/kicad/BKM-10Rp2040 v2.kicad_pcb (KiCad board)
At the start: 2 copper layers, 34.3 x 77.2 mm, 11 parts, among them J1 DB9_Female_MountingHoles, J2 Conn_01x04, SW1 SW_DPST_x2, U1 ADM3063EARZ-ND, U2 Pico, U3 TSOP335xx

Commit message: fix display on SH1106
Changed lines of the file:
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@@
       (drillshape 0)
       (scaleselection 1)
-      (outputdirectory "gerbers"))
+      (outputdirectory "gerbers/"))
   )
   (net 0 "")
@@
       (effects (font (size 0.5 0.5) (thickness 0.08)))
     )
-    (pad 2 smd roundrect (at 1.0375 0 180) (size 1.175 1.45) (layers F.Cu F.Paste F.Mask) (roundrect_rratio 0.212766)
+    (pad 2 smd roundrect (at 1.0375 0 180) (size 1.175 1.45) (layers F.Cu F.Paste F.Mask) (roundrect_rratio 0.2127659574468085)
       (net 29 GND))
-    (pad 1 smd roundrect (at -1.0375 0 180) (size 1.175 1.45) (layers F.Cu F.Paste F.Mask) (roundrect_rratio 0.212766)
+    (pad 1 smd roundrect (at -1.0375 0 180) (size 1.175 1.45) (layers F.Cu F.Paste F.Mask) (roundrect_rratio 0.2127659574468085)
       (net 28 +5V))
     (model ${KISYS3DMOD}/Capacitor_SMD.3dshapes/C_0805_2012Metric.wrl
@@
       (effects (font (size 0.5 0.5) (thickness 0.08)))
     )
-    (pad 2 smd roundrect (at 1.0375 0 90) (size 1.175 1.45) (layers F.Cu F.Paste F.Mask) (roundrect_rratio 0.212766)
+    (pad 2 smd roundrect (at 1.0375 0 90) (size 1.175 1.45) (layers F.Cu F.Paste F.Mask) (roundrect_rratio 0.2127659574468085)
       (net 28 +5V))
-    (pad 1 smd roundrect (at -1.0375 0 90) (size 1.175 1.45) (layers F.Cu F.Paste F.Mask) (roundrect_rratio 0.212766)
+    (pad 1 smd roundrect (at -1.0375 0 90) (size 1.175 1.45) (layers F.Cu F.Paste F.Mask) (roundrect_rratio 0.2127659574468085)
       (net 29 GND))
     (model ${KISYS3DMOD}/Capacitor_SMD.3dshapes/C_0805_2012Metric.wrl
@@
       (effects (font (size 0.8 0.8) (thickness 0.12)))
     )
-    (pad 2 smd roundrect (at 1.55 0 180) (size 1.3 1.75) (layers F.Cu F.Paste F.Mask) (roundrect_rratio 0.1923076923076923)
+    (pad 2 smd roundrect (at 1.55 0 180) (size 1.3 1.75) (layers F.Cu F.Paste F.Mask) (roundrect_rratio 0.1923069230769231)
       (net 31 TXD+))
-    (pad 1 smd roundrect (at -1.55 0 180) (size 1.3 1.75) (layers F.Cu F.Paste F.Mask) (roundrect_rratio 0.1923076923076923)
+    (pad 1 smd roundrect (at -1.55 0 180) (size 1.3 1.75) (layers F.Cu F.Paste F.Mask) (roundrect_rratio 0.1923069230769231)
       (net 33 TXD-))
     (model ${KISYS3DMOD}/Resistor_SMD.3dshapes/R_1206_3216Metric.wrl

Commit message: add new case models
Connections:
- net ~RE~ renamed ~{RE}
Other:
- net class Default removed
